Commit message: URDF fixed

File: adventure_simulator/adventure_description/finn/finn.urdf.xacro (robot description, xacro)
@@ -8,5 +8,5 @@
   <xacro:include filename="$(find adventure_description)/urdf/sensors/asus_xtion_pro.urdf.xacro"/>
   <xacro:sensor_asus_xtion_pro parent="base_link">
-    <origin xyz="${0.0} 0.0 0.20" rpy="0.0 0.0 0.0"/>
+    <origin xyz="${0.14} 0.02 0.1" rpy="0.0 0.0 0.0"/>
   </xacro:sensor_asus_xtion_pro>
   <!-- Generic camera

Commit message: Minor URDF fix

File: adventure_simulator/adventure_description/finn/finn.urdf.xacro (robot description, xacro)
@@ -8,5 +8,5 @@
   <xacro:include filename="$(find adventure_description)/urdf/sensors/asus_xtion_pro.urdf.xacro"/>
   <xacro:sensor_asus_xtion_pro parent="base_link">
-    <origin xyz="${0.14} 0.02 0.1" rpy="0.0 0.0 0.0"/>
+    <origin xyz="${0.14} -0.02 0.1" rpy="3.14 0.0 0.0"/>
   </xacro:sensor_asus_xtion_pro>
   <!-- Generic camera
